Commit message: 1 - drawing whole robot 2 - bug: some positions are off center - joint

File: data/my2wr.xacro (robot description, xacro)
@@ -65,5 +65,5 @@
     </collision>
     <visual>
-      <origin rpy="0 0 0" xyz="0 0 0"/>
+      <origin rpy="0 0 0" xyz="0 0 0.1"/>
       <geometry>
         <box size="0.5 0.3 0.07"/>
@@ -112,4 +112,5 @@
         <cylinder length="0.04" radius="0.1"/>
       </geometry>
+      <material name="red"/>
     </visual>
   </link>
@@ -139,4 +140,5 @@
         <cylinder length="0.04" radius="0.1"/>
       </geometry>
+      <material name="red"/>
     </visual>
   </link>
