Commit message: 1 - corrected wavefront objects to be 1m in scale 2 - added wavefront mesh loading and display 3 - colour is now loaded from urdf file

File: data/nas_robot_latest.xacro (robot description, xacro)
@@ -6,12 +6,27 @@
   <xacro:property name="rkolesa" value="0.2"/>
   <xacro:property name="hkolesa" value="0.1"/>
-  <material name="oranzova">
-    <color rgba="1 0.65 0 1"/>
-  </material>
-  <material name="cervena">
-    <color rgba="1 0 0 1"/>
-  </material>
-  <material name="biela">
-    <color rgba="1 1 1 1"/>
+  <material name="black">
+    <color rgba="0.0 0.0 0.0 1.0"/>
+  </material>
+  <material name="blue">
+    <color rgba="0.203125 0.23828125 0.28515625 1.0"/>
+  </material>
+  <material name="green">
+    <color rgba="0.0 0.8 0.0 1.0"/>
+  </material>
+  <material name="grey">
+    <color rgba="0.2 0.2 0.2 1.0"/>
+  </material>
+  <material name="orange">
+    <color rgba="1.0 0.423529411765 0.0392156862745 1.0"/>
+  </material>
+  <material name="brown">
+    <color rgba="0.870588235294 0.811764705882 0.764705882353 1.0"/>
+  </material>
+  <material name="red">
+    <color rgba="0.80078125 0.12890625 0.1328125 1.0"/>
+  </material>
+  <material name="white">
+    <color rgba="1.0 1.0 1.0 1.0"/>
   </material>
   <!-- umoznenie ovladania -->
@@ -44,5 +59,5 @@
         <box size="${dlzka} ${sirka} ${vyska}"/>
       </geometry>
-      <material name="oranzova"/>
+      <material name="orange"/>
     </visual>
     <collision name='telo_collision'>
@@ -67,4 +82,5 @@
         <sphere radius="0.05"/>
       </geometry>
+      <material name="blue"/>
     </visual>
     <collision name='vsesmerove_collision'>
@@ -99,5 +115,5 @@
           <cylinder radius="0.1" length="0.05"/>
         </geometry>
-        <material name="biela"/>
+        <material name="white"/>
       </visual>
       <collision name="${prefix}_koleso_collision">
@@ -176,5 +192,5 @@
         <box size="0.05 0.05 0.02"/>
       </geometry>
-      <material name="cervena"/>
+      <material name="red"/>
     </visual>
     <collision>

Commit message: 1 - objects are now ready to be drawn in opengl 2 - minor improvements

File: data/nas_robot_latest.xacro (robot description, xacro)
@@ -55,5 +55,5 @@
     <!--pose>0 0 0.1 0 0 0</pose-->
     <visual name='telo_visual'>
-      <origin xyz="0 0 0" rpy=" 0 0 0"/>
+      <origin xyz="0 0 0" rpy="0 0 0"/>
       <geometry>
         <box size="${dlzka} ${sirka} ${vyska}"/>
@@ -68,5 +68,5 @@
     <inertial>
       <mass value="10.0"/>
-      <origin xyz="0.0 0 0.1" rpy=" 0 0 0"/>
+      <origin xyz="0.0 0 0.1" rpy="0 0 0"/>
       <inertia
               ixx="0.5" ixy="0" ixz="0"
@@ -78,5 +78,5 @@
   <link name="vsesmerove_koleso">
     <visual name='vsesmerove_visual'>
-      <origin xyz="-0.15 0 -0.05" rpy=" 0 0 0"/>
+      <origin xyz="-0.15 0 -0.05" rpy="0 0 0"/>
       <geometry>
         <sphere radius="0.05"/>
@@ -85,5 +85,5 @@
     </visual>
     <collision name='vsesmerove_collision'>
-      <origin xyz="-0.15 0 -0.05" rpy=" 0 0 0"/>
+      <origin xyz="-0.15 0 -0.05" rpy="0 0 0"/>
       <geometry>
         <sphere radius="0.05"/>

Commit message: 1 - robot now displays correctly

File: data/nas_robot_latest.xacro (robot description, xacro)
@@ -55,5 +55,5 @@
     <!--pose>0 0 0.1 0 0 0</pose-->
     <visual name='telo_visual'>
-      <origin xyz="0 0 0" rpy="0 0 0"/>
+      <origin xyz="0 0 0.1" rpy="0 0 0"/>
       <geometry>
         <box size="${dlzka} ${sirka} ${vyska}"/>
@@ -115,5 +115,5 @@
           <cylinder radius="0.1" length="0.05"/>
         </geometry>
-        <material name="white"/>
+        <material name="red"/>
       </visual>
       <collision name="${prefix}_koleso_collision">

Commit message: 1 - pyQt6 windowing 2 - GUI added

File: data/nas_robot_latest.xacro (robot description, xacro)
@@ -78,5 +78,5 @@
   <link name="vsesmerove_koleso">
     <visual name='vsesmerove_visual'>
-      <origin xyz="-0.15 0 -0.05" rpy="0 0 0"/>
+      <origin xyz="-0.15 0 -0.1" rpy="0 0 0"/>
       <geometry>
         <sphere radius="0.05"/>

Commit message: 1 - added kinematics and movement

File: data/nas_robot_latest.xacro (robot description, xacro)
@@ -4,6 +4,6 @@
   <xacro:property name="sirka" value="0.2"/>
   <xacro:property name="vyska" value="0.1"/>
-  <xacro:property name="rkolesa" value="0.2"/>
-  <xacro:property name="hkolesa" value="0.1"/>
+  <xacro:property name="rkolesa" value="0.1"/>
+  <xacro:property name="hkolesa" value="0.05"/>
   <material name="black">
     <color rgba="0.0 0.0 0.0 1.0"/>
@@ -78,5 +78,5 @@
   <link name="vsesmerove_koleso">
     <visual name='vsesmerove_visual'>
-      <origin xyz="-0.15 0 -0.1" rpy="0 0 0"/>
+      <origin xyz="0 0 0" rpy="0 0 0"/>
       <geometry>
         <sphere radius="0.05"/>
@@ -103,5 +103,5 @@
   </link>
   <joint name="vsesmerove_koleso_upevnenie" type="fixed">
-    <origin xyz="-0.1 0 0.05" rpy="0 0 0"/>
+    <origin xyz="-0.15 0 -0.05" rpy="0 0 0"/>
     <parent link="telo"/>
     <child link="vsesmerove_koleso"/>
@@ -113,5 +113,5 @@
         <origin xyz="0 0 0" rpy="0 1.5707 1.5707"/>
         <geometry>
-          <cylinder radius="0.1" length="0.05"/>
+          <cylinder radius="${rkolesa}" length="${hkolesa}"/>
         </geometry>
         <material name="red"/>
@@ -120,5 +120,5 @@
         <origin xyz="0 0 0" rpy="0 1.5707 1.5707"/>
         <geometry>
-          <cylinder radius="0.1" length="0.05"/>
+          <cylinder radius="${rkolesa}" length="${hkolesa}"/>
         </geometry>
       </collision>
@@ -145,5 +145,5 @@
 -->
     <joint type="continuous" name="${prefix}_koleso_zaves">
-      <origin xyz="0.1 ${reflect*0.15} 0" rpy="0 0 0"/>
+      <origin xyz="0.1 ${reflect*0.125} 0" rpy="0 0 0"/>
       <child link="${prefix}_koleso"/>
       <parent link="telo"/>
