Commit message: 1 - camera follows robot 2 - texture on ground

File: data/differential_drive.xacro (robot description, xacro)
@@ -150,5 +150,5 @@
   </link>
   <joint name="nas_lidar_upevnenie" type="fixed">
-    <origin xyz="0.1 0 0.1" rpy="0 0 0"/>
+    <origin xyz="0.1 0 0.06" rpy="0 0 0"/>
     <parent link="telo"/>
     <child link="nas_lidar"/>
